Commit message: fix jackal description

File: jackal_description/urdf/accessories/d435.urdf.xacro (robot description, xacro)
@@ -53,5 +53,5 @@
         <origin xyz="${d435_zero_depth_to_glass + d435_glass_to_front} ${-d435_cam_depth_py} 0" rpy="${M_PI/2} 0 ${M_PI/2}"/>
         <geometry>
-          <mesh filename="file://$(find husky_description)/meshes/d435.dae" />
+          <mesh filename="file://$(find jackal_description)/meshes/d435.dae" />
         </geometry>
       </xacro:if>

Commit message: isaac sim

File: jackal_description/urdf/accessories/d435.urdf.xacro (robot description, xacro)
@@ -53,5 +53,5 @@
         <origin xyz="${d435_zero_depth_to_glass + d435_glass_to_front} ${-d435_cam_depth_py} 0" rpy="${M_PI/2} 0 ${M_PI/2}"/>
         <geometry>
-          <mesh filename="file://$(find jackal_description)/meshes/d435.dae" />
+          <mesh filename="package://jackal_description/meshes/d435.dae"/>
         </geometry>
       </xacro:if>

File: jackal_description/urdf/jackal.urdf.xacro (robot description, xacro)
@@ -228,5 +228,12 @@
     <hardware>
       <xacro:if value="$(arg is_sim)">
-        <plugin>gazebo_ros2_control/GazeboSystem</plugin>
+        <xacro:if value="$(arg isaac_sim)">
+            <plugin>topic_based_ros2_control/TopicBasedSystem</plugin>
+            <param name="joint_commands_topic">/isaac_joint_commands</param>
+            <param name="joint_states_topic">/isaac_joint_states</param>
+        </xacro:if>
+        <xacro:unless value="$(arg isaac_sim)">
+            <plugin>gazebo_ros2_control/GazeboSystem</plugin>
+        </xacro:unless>
       </xacro:if>
       <xacro:unless value="$(arg is_sim)">
