Commit message: imu noise and minor fixes

File: jackal_description/urdf/accessories/hokuyo_ust10.urdf.xacro (robot description, xacro)
@@ -2,5 +2,5 @@
 <robot xmlns:xacro="http://ros.org/wiki/xacro">
   <xacro:macro name="hokuyo_ust10_mount" params="prefix topic parent_link *origin">
-    <xacro:macro name="hokuyo_ust10" params="frame:=laser topic:=scan sample_size:=720 update_rate:=50
+    <xacro:macro name="hokuyo_ust10" params="frame:=laser topic:=scan sample_size:=720 update_rate:=30
                min_angle:=-2.35619 max_angle:=2.35619 min_range:=0.1 max_range:=30.0 robot_namespace:=/">
       <link name="${frame}">
@@ -14,5 +14,4 @@
       </link>
       <gazebo reference="${frame}">
-        <turnGravityOff>true</turnGravityOff>
         <sensor type="ray" name="${frame}">
           <pose>0 0 0 0 0 0</pose>
@@ -36,5 +35,5 @@
               <type>gaussian</type>
               <mean>0.0</mean>
-              <stddev>0.001</stddev>
+              <stddev>0.01</stddev>
             </noise>
           </ray>

Commit message: gazebo pose3d

File: jackal_description/urdf/accessories/hokuyo_ust10.urdf.xacro (robot description, xacro)
@@ -2,5 +2,5 @@
 <robot xmlns:xacro="http://ros.org/wiki/xacro">
   <xacro:macro name="hokuyo_ust10_mount" params="prefix topic parent_link *origin">
-    <xacro:macro name="hokuyo_ust10" params="frame:=laser topic:=scan sample_size:=720 update_rate:=30
+    <xacro:macro name="hokuyo_ust10" params="frame:=laser topic:=scan sample_size:=360 update_rate:=30
                min_angle:=-3.1416 max_angle:=3.1416 min_range:=0.1 max_range:=30.0 robot_namespace:=/">
       <link name="${frame}">
@@ -14,5 +14,5 @@
       </link>
       <gazebo reference="${frame}">
-        <sensor type="ray" name="${frame}">
+        <sensor type="gpu_ray" name="${frame}">
           <pose>0 0 0 0 0 0</pose>
           <visualize>false</visualize>
