Commit message: push to humble

File: jackal_description/urdf/accessories.urdf.xacro (robot description, xacro)
@@ -118,5 +118,5 @@
     <!-- Velodyne VLP16 -->
     <xacro:if value="${lidar_3d_model == 'vlp16'}">
-      <xacro:vlp16_mount topic="${topic}" tower="${tower}" prefix="${prefix}" parent_link="${parent}" >
+      <xacro:vlp16_mount topic="${topic}" tower="${tower}" prefix="${prefix}" parent_link="${parent}">
         <origin xyz="$(optenv JACKAL_LASER_3D_OFFSET 0 0 0)" rpy="$(optenv JACKAL_LASER_3D_RPY 0 0 0)" />
       </xacro:vlp16_mount>
@@ -124,5 +124,5 @@
     <!-- Velodyne HDL-32E -->
     <xacro:if value="${lidar_3d_model == 'hdl32e'}">
-      <xacro:hdl32e_mount topic="${topic}" tower="${tower}" prefix="${prefix}" parent_link="${parent}" >
+      <xacro:hdl32e_mount topic="${topic}" tower="${tower}" prefix="${prefix}" parent_link="${parent}">
         <origin xyz="$(optenv JACKAL_LASER_3D_OFFSET 0 0 0)" rpy="$(optenv JACKAL_LASER_3D_RPY 0 0 0)" />
       </xacro:hdl32e_mount>
@@ -192,4 +192,5 @@
   <!--
     Add Cameras.
+    - JACKAL_D435
     - JACKAL_FLEA3
     - JACKAL_STEREO_FLEA3
@@ -199,4 +200,15 @@
   <xacro:include filename="$(find jackal_description)/urdf/accessories/camera_mount.urdf.xacro" />
   <!--xacro:include filename="$(find pointgrey_camera_description)/urdf/pointgrey_flea3.urdf.xacro" /-->
+  <!-- If enabled, generate the d435 camera payload. -->
+  <xacro:if value="$(optenv JACKAL_D435 0)">
+    <xacro:property name="name" value="$(optenv JACKAL_D435_NAME front)" />
+    <xacro:property name="mount" value="$(optenv JACKAL_D435_MOUNT front)" />
+    <xacro:property name="camera_xyz" default="$(optenv JACKALD435_XYZ 0.042 0.0 0.0)" />
+    <xacro:property name="camera_rpy" default="$(optenv JACKALD435_RPY 0.0 0.0 0.0)" />
+    <xacro:property name="prefix" value="$(optenv JACKAL_D435_PREFIX ${mount})" />
+    <xacro:property name="parent" value="$(optenv JACKAL_D435_PARENT ${mount}_mount)" />
+    <xacro:property name="camera_frame_id" value="$(optenv JACKAL_D435_FRAME camera_color_frame)" />
+    <xacro:include filename="$(find jackal_description)/urdf/accessories/d435.urdf.xacro" />
+  </xacro:if>
   <!-- If enabled, generate the flea3 camera payload with a tilt of 30 degrees. -->
   <xacro:if value="$(optenv JACKAL_FLEA3 0)">
@@ -207,13 +219,10 @@
     <xacro:property name="prefix" value="$(optenv JACKAL_FLEA3_PREFIX ${mount})" />
     <xacro:property name="parent" value="$(optenv JACKAL_FLEA3_PARENT ${mount}_mount)" />
-    <xacro:pointgrey_flea3 frame="${prefix}_camera" name="${name}"
-      camera_x="0.0754" camera_y="0.029" camera_z="0.029"
-      camera_mass="0.085" hfov="1.0471975512" fps="60" width="640" height="512"/>
+    <xacro:pointgrey_flea3 frame="${prefix}_camera" name="${name}" camera_x="0.0754" camera_y="0.029" camera_z="0.029" camera_mass="0.085" hfov="1.0471975512" fps="60" width="640" height="512"/>
     <!-- Mount Enabled -->
     <xacro:if value="${tower}">
       <xacro:camera_mount prefix="${prefix}" tilt="${tilt}"/>
       <joint name="${prefix}_camera_mount_joint" type="fixed">
-        <origin xyz="$(optenv JACKAL_FLEA3_OFFSET 0 0 0)"
-                rpy="$(optenv JACKAL_FLEA3_RPY 0 0 0)" />
+        <origin xyz="$(optenv JACKAL_FLEA3_OFFSET 0 0 0)" rpy="$(optenv JACKAL_FLEA3_RPY 0 0 0)" />
         <parent link="${parent}" />
         <child link="${prefix}_camera_mount" />
@@ -229,12 +238,10 @@
       <link name="${prefix}_camera_base"/>
       <joint name="${prefix}_camera_base_joint" type="fixed">
-        <origin xyz="$(optenv JACKAL_FLEA3_OFFSET 0 0 0)"
-                rpy="$(optenv JACKAL_FLEA3_RPY 0 0 0)" />
+        <origin xyz="$(optenv JACKAL_FLEA3_OFFSET 0 0 0)" rpy="$(optenv JACKAL_FLEA3_RPY 0 0 0)" />
         <parent link="${parent}" />
         <child link="${prefix}_camera_base" />
       </joint>
       <joint name="${prefix}_camera_joint" type="fixed">
-        <origin xyz="0 0 0.0145"
-                rpy="0 0 0" />
+        <origin xyz="0 0 0.0145" rpy="0 0 0" />
         <parent link="${prefix}_camera_base" />
         <child link="${prefix}_camera" />
@@ -255,12 +262,9 @@
     <xacro:stereo_camera_mount prefix="${prefix}" tilt="${tilt}"/>
     <joint name="${prefix}_stereo_camera_mount_joint" type="fixed">
-      <origin xyz="$(optenv JACKAL_FLEA3_OFFSET 0 0 0)"
-              rpy="$(optenv JACKAL_FLEA3_RPY 0 0 0)" />
+      <origin xyz="$(optenv JACKAL_FLEA3_OFFSET 0 0 0)" rpy="$(optenv JACKAL_FLEA3_RPY 0 0 0)" />
       <parent link="${parent}" />
       <child link="${prefix}_stereo_camera_mount" />
     </joint>
-    <xacro:pointgrey_flea3 frame="${prefix}_left_camera" name="${left_name}"
-      camera_x="0.0754" camera_y="0.029" camera_z="0.029"
-      camera_mass="0.085" hfov="1.0471975512" fps="60" width="640" height="512"/>
+    <xacro:pointgrey_flea3 frame="${prefix}_left_camera" name="${left_name}" camera_x="0.0754" camera_y="0.029" camera_z="0.029" camera_mass="0.085" hfov="1.0471975512" fps="60" width="640" height="512"/>
     <joint name="${prefix}_left_stereo_camera_bracket_joint" type="fixed">
       <origin xyz="0.015 ${separation} 0.0599" rpy="0 0 0" />
@@ -268,7 +272,5 @@
       <child link="${prefix}_left_camera" />
     </joint>
-    <xacro:pointgrey_flea3 frame="${prefix}_right_camera" name="${right_name}"
-      camera_x="0.0754" camera_y="0.029" camera_z="0.029"
-      camera_mass="0.085" hfov="1.0471975512" fps="60" width="640" height="512"/>
+    <xacro:pointgrey_flea3 frame="${prefix}_right_camera" name="${right_name}" camera_x="0.0754" camera_y="0.029" camera_z="0.029" camera_mass="0.085" hfov="1.0471975512" fps="60" width="640" height="512"/>
     <joint name="${prefix}_right_stereo_camera_bracket_joint" type="fixed">
       <origin xyz="0.015 -${separation} 0.0599" rpy="0 0 0" />
@@ -293,6 +295,5 @@
       <xacro:camera_mount prefix="${prefix}" tilt="${tilt}"/>
       <joint name="${prefix}_camera_mount_joint" type="fixed">
-        <origin xyz="$(optenv JACKAL_BB2_OFFSET 0 0 0)"
-                rpy="$(optenv JACKAL_BB2_RPY 0 0 0)" />
+        <origin xyz="$(optenv JACKAL_BB2_OFFSET 0 0 0)" rpy="$(optenv JACKAL_BB2_RPY 0 0 0)" />
         <parent link="${parent}" />
         <child link="${prefix}_camera_mount" />
@@ -308,6 +309,5 @@
       <link name="${prefix}_camera_base" type="fixed"/>
       <joint name="${prefix}_camera_base_joint" type="fixed">
-        <origin xyz="$(optenv JACKAL_BB2_OFFSET 0 0 0)"
-                rpy="$(optenv JACKAL_BB2_RPY 0 0 0)" />
+        <origin xyz="$(optenv JACKAL_BB2_OFFSET 0 0 0)" rpy="$(optenv JACKAL_BB2_RPY 0 0 0)" />
         <parent link="${parent}" />
         <child link="${prefix}_camera_base" />
@@ -324,10 +324,5 @@
     <xacro:include filename="$(find jackal_description)/urdf/accessories/hokuyo_ust10.urdf.xacro" />
     <xacro:if value="$(optenv JACKAL_FRONT_FENDER_UST10 0)">
-      <xacro:hokuyo_ust10_mount
-        prefix="front"
-        parent_link="front_fender_accessory_link"
-        min_angle="${-pi/2}"
-        max_angle="${pi/2}"
-        topic="$(optenv JACKAL_FRONT_LASER_TOPIC front/scan)">
+      <xacro:hokuyo_ust10_mount prefix="front" parent_link="front_fender_accessory_link" min_angle="${-pi/2}" max_angle="${pi/2}" topic="$(optenv JACKAL_FRONT_LASER_TOPIC front/scan)">
         <origin xyz="0 0 0" rpy="0 0 0" />
       </xacro:hokuyo_ust10_mount>
@@ -336,10 +331,5 @@
   <xacro:if value="$(optenv JACKAL_REAR_ACCESSORY_FENDER 0)">
     <xacro:if value="$(optenv JACKAL_REAR_FENDER_UST10 0)">
-      <xacro:hokuyo_ust10_mount
-        prefix="rear"
-        parent_link="rear_fender_accessory_link"
-        min_angle="${-pi/2}"
-        max_angle="${pi/2}"
-        topic="$(optenv JACKAL_REAR_LASER_TOPIC rear/scan)">
+      <xacro:hokuyo_ust10_mount prefix="rear" parent_link="rear_fender_accessory_link" min_angle="${-pi/2}" max_angle="${pi/2}" topic="$(optenv JACKAL_REAR_LASER_TOPIC rear/scan)">
         <origin xyz="0 0 0" rpy="0 0 0" />
       </xacro:hokuyo_ust10_mount>

Commit message: d435 stereo

File: jackal_description/urdf/accessories.urdf.xacro (robot description, xacro)
@@ -210,4 +210,15 @@
     <xacro:property name="camera_frame_id" value="$(optenv JACKAL_D435_FRAME camera_color_frame)" />
     <xacro:include filename="$(find jackal_description)/urdf/accessories/d435.urdf.xacro" />
+  </xacro:if>
+  <!-- If enabled, generate the d435 camera payload. -->
+  <xacro:if value="$(optenv JACKAL_D435_STEREO 0)">
+    <xacro:property name="name" value="$(optenv JACKAL_D435_STEREO_NAME front)" />
+    <xacro:property name="mount" value="$(optenv JACKAL_D435_STEREO_MOUNT front)" />
+    <xacro:property name="camera_xyz" default="$(optenv JACKAL_D435_STEREO_XYZ 0.042 0.0 0.0)" />
+    <xacro:property name="camera_rpy" default="$(optenv JACKAL_D435_STEREO_RPY 0.0 0.0 0.0)" />
+    <xacro:property name="prefix" value="$(optenv JACKAL_D435_STEREO_PREFIX ${mount})" />
+    <xacro:property name="parent" value="$(optenv JACKAL_D435_STEREO_PARENT ${mount}_mount)" />
+    <xacro:property name="camera_frame_id" value="$(optenv JACKAL_D435_STEREO_FRAME camera_infra1_frame)" />
+    <xacro:include filename="$(find jackal_description)/urdf/accessories/d435_stereo.urdf.xacro" />
   </xacro:if>
   <!-- If enabled, generate the flea3 camera payload with a tilt of 30 degrees. -->

File: jackal_description/urdf/accessories/hokuyo_ust10.urdf.xacro (robot description, xacro)
@@ -3,5 +3,5 @@
   <xacro:macro name="hokuyo_ust10_mount" params="prefix topic parent_link *origin">
     <xacro:macro name="hokuyo_ust10" params="frame:=laser topic:=scan sample_size:=720 update_rate:=30
-               min_angle:=-2.35619 max_angle:=2.35619 min_range:=0.1 max_range:=30.0 robot_namespace:=/">
+               min_angle:=-3.1416 max_angle:=3.1416 min_range:=0.1 max_range:=30.0 robot_namespace:=/">
       <link name="${frame}">
         <inertial>

Commit message: stereo camera description

File: jackal_description/urdf/accessories.urdf.xacro (robot description, xacro)
@@ -201,5 +201,7 @@
   <!--xacro:include filename="$(find pointgrey_camera_description)/urdf/pointgrey_flea3.urdf.xacro" /-->
   <!-- If enabled, generate the d435 camera payload. -->
-  <xacro:if value="$(optenv JACKAL_D435 0)">
+  <xacro:property name="d435" value="$(optenv JACKAL_D435 0)" />
+  <xacro:property name="d435_stereo" value="$(optenv JACKAL_D435 0)" />
+  <xacro:if value="${d435 or d435_stereo}">
     <xacro:property name="name" value="$(optenv JACKAL_D435_NAME front)" />
     <xacro:property name="mount" value="$(optenv JACKAL_D435_MOUNT front)" />
@@ -209,16 +211,6 @@
     <xacro:property name="parent" value="$(optenv JACKAL_D435_PARENT ${mount}_mount)" />
     <xacro:property name="camera_frame_id" value="$(optenv JACKAL_D435_FRAME camera_color_frame)" />
+    <xacro:property name="stereo_camera_frame_id" value="$(optenv JACKAL_D435_STEREO_FRAME camera_infra1_frame)" />
     <xacro:include filename="$(find jackal_description)/urdf/accessories/d435.urdf.xacro" />
-  </xacro:if>
-  <!-- If enabled, generate the d435 camera payload. -->
-  <xacro:if value="$(optenv JACKAL_D435_STEREO 0)">
-    <xacro:property name="name" value="$(optenv JACKAL_D435_STEREO_NAME front)" />
-    <xacro:property name="mount" value="$(optenv JACKAL_D435_STEREO_MOUNT front)" />
-    <xacro:property name="camera_xyz" default="$(optenv JACKAL_D435_STEREO_XYZ 0.042 0.0 0.0)" />
-    <xacro:property name="camera_rpy" default="$(optenv JACKAL_D435_STEREO_RPY 0.0 0.0 0.0)" />
-    <xacro:property name="prefix" value="$(optenv JACKAL_D435_STEREO_PREFIX ${mount})" />
-    <xacro:property name="parent" value="$(optenv JACKAL_D435_STEREO_PARENT ${mount}_mount)" />
-    <xacro:property name="camera_frame_id" value="$(optenv JACKAL_D435_STEREO_FRAME camera_infra1_frame)" />
-    <xacro:include filename="$(find jackal_description)/urdf/accessories/d435_stereo.urdf.xacro" />
   </xacro:if>
   <!-- If enabled, generate the flea3 camera payload with a tilt of 30 degrees. -->

File: jackal_description/urdf/accessories/d435.urdf.xacro (robot description, xacro)
@@ -133,31 +133,89 @@
   </xacro:if>
   <xacro:if value="$(arg is_sim)">
-    <gazebo reference="${camera_frame_id}">
-      <sensor type="depth" name="d435">
-        <always_on>1</always_on>
-        <update_rate>30</update_rate>
-        <camera name="camera">
-          <horizontal_fov>${60*3.14/180.0}</horizontal_fov>
-          <image>
-            <format>R8G8B8</format>
-            <width>640</width>
-            <height>480</height>
-          </image>
-          <clip>
-            <near>0.15</near>
-            <far>10.0</far>
-          </clip>
-        </camera>
-        <plugin name="camera_plugin" filename="libgazebo_ros_camera.so">
-          <ros>
-          </ros>
-          <!-- Set camera name. If empty, defaults to sensor name (i.e. "sensor_name") -->
-          <camera_name>camera</camera_name>
-          <!-- Set TF frame name. If empty, defaults to link name (i.e. "link_name") -->
-          <frame_name>camera_color_optical_frame</frame_name>
-          <!--hack_baseline>0.07</hack_baseline-->
-        </plugin>
-      </sensor>
-    </gazebo>
+    <!-- CAMERA PLUGIN GAZEBO -->
+    <xacro:if value="$(optenv JACKAL_D435 0)">
+      <gazebo reference="${camera_frame_id}">
+        <sensor type="depth" name="d435">
+          <always_on>1</always_on>
+          <update_rate>30</update_rate>
+          <camera name="camera">
+            <horizontal_fov>${60*3.14/180.0}</horizontal_fov>
+            <image>
+              <format>R8G8B8</format>
+              <width>640</width>
+              <height>480</height>
+            </image>
+            <clip>
+              <near>0.15</near>
+              <far>10.0</far>
+            </clip>
+          </camera>
+          <plugin name="camera_plugin" filename="libgazebo_ros_camera.so">
+            <!-- Set camera name. If empty, defaults to sensor name (i.e. "sensor_name") -->
+            <camera_name>camera</camera_name>
+            <!-- Set TF frame name. If empty, defaults to link name (i.e. "link_name") -->
+            <frame_name>camera_color_optical_frame</frame_name>
+          </plugin>
+        </sensor>
+      </gazebo>
+    </xacro:if>
+    <!-- MULTICAMERA PLUGIN GAZEBO -->
+    <xacro:if value="$(optenv JACKAL_D435_STEREO 0)">
+      <!-- Both cameras in the pair are anchored off the left camera frame. -->
+      <gazebo reference="${stereo_camera_frame_id}">
+        <sensor type="multicamera" name="d435_stereo">
+          <always_on>1</always_on>
+          <update_rate>30</update_rate>
+          <camera name="left">
+            <horizontal_fov>${60*3.14/180.0}</horizontal_fov>
+            <image>
+              <format>R8G8B8</format>
+              <width>640</width>
+              <height>480</height>
+            </image>
+            <clip>
+              <near>0.15</near>
+              <far>25.0</far>
+            </clip>
+            <noise>
+              <type>gaussian</type>
+              <!-- Noise is sampled independently per pixel on each frame.
+                  That pixel's noise value is added to each of its color
+                  channels, which at that point lie in the range [0,1]. -->
+              <mean>0.0</mean>
+              <stddev>0.0001</stddev>
+          </noise>
+          </camera>
+          <camera name="right">
+          <pose>0 -0.07 0 0 0 0</pose>
+            <horizontal_fov>${60*3.14/180.0}</horizontal_fov>
+            <image>
+              <format>R8G8B8</format>
+              <width>640</width>
+              <height>480</height>
+            </image>
+            <clip>
+              <near>0.15</near>
+              <far>25.0</far>
+            </clip>
+            <noise>
+              <type>gaussian</type>
+              <!-- Noise is sampled independently per pixel on each frame.
+                  That pixel's noise value is added to each of its color
+                  channels, which at that point lie in the range [0,1]. -->
+              <mean>0.0</mean>
+              <stddev>0.0001</stddev>
+          </noise>
+          </camera>
+          <plugin name="stereo_camera_plugin" filename="libgazebo_ros_camera.so">
+            <!-- Set camera name. If empty, defaults to sensor name (i.e. "sensor_name") -->
+            <camera_name>camera_stereo</camera_name>
+            <!-- Set TF frame name. If empty, defaults to link name (i.e. "link_name") -->
+            <frame_name>camera_infra1_optical_frame</frame_name>
+            <hack_baseline>0.05</hack_baseline>
+          </plugin>
+        </sensor>
+      </gazebo>
+    </xacro:if>
   </xacro:if>
 </robot>

Commit message: fix on minor parameters

File: jackal_description/urdf/accessories.urdf.xacro (robot description, xacro)
@@ -202,5 +202,5 @@
   <!-- If enabled, generate the d435 camera payload. -->
   <xacro:property name="d435" value="$(optenv JACKAL_D435 0)" />
-  <xacro:property name="d435_stereo" value="$(optenv JACKAL_D435 0)" />
+  <xacro:property name="d435_stereo" value="$(optenv JACKAL_D435_STEREO 0)" />
   <xacro:if value="${d435 or d435_stereo}">
     <xacro:property name="name" value="$(optenv JACKAL_D435_NAME front)" />
