Commit message: add env-hooks to export env variables

File: jackal_description/urdf/jackal.urdf.xacro (robot description, xacro)
@@ -16,32 +16,40 @@
   <xacro:property name="chassis_width" value="0.310" />
   <xacro:property name="chassis_height" value="0.184" />
-  <xacro:property name="dummy_inertia" value="1e-09"/>
+  <xacro:property name="dummy_inertia" value="1e-09" />
   <xacro:property name="mount_spacing" value="0.120" />
-  <material name="dark_grey"><color rgba="0.2 0.2 0.2 1.0" /></material>
-  <material name="light_grey"><color rgba="0.4 0.4 0.4 1.0" /></material>
-  <material name="yellow"><color rgba="0.8 0.8 0.0 1.0" /></material>
-  <material name="black"><color rgba="0.15 0.15 0.15 1.0" /></material>
+  <material name="dark_grey">
+    <color rgba="0.2 0.2 0.2 1.0" />
+  </material>
+  <material name="light_grey">
+    <color rgba="0.4 0.4 0.4 1.0" />
+  </material>
+  <material name="yellow">
+    <color rgba="0.8 0.8 0.0 1.0" />
+  </material>
+  <material name="black">
+    <color rgba="0.15 0.15 0.15 1.0" />
+  </material>
   <xacro:macro name="wheel" params="prefix *joint_pose">
     <link name="${prefix}_wheel_link">
       <visual>
-        <origin xyz="0 0 0" rpy="${PI/2} 0 0"/>
-        <geometry>
-          <mesh filename="package://jackal_description/meshes/jackal-wheel.stl"/>
+        <origin xyz="0 0 0" rpy="${PI/2} 0 0" />
+        <geometry>
+          <mesh filename="package://jackal_description/meshes/jackal-wheel.stl" />
         </geometry>
         <material name="black" />
       </visual>
       <collision>
-        <origin xyz="0 0 0" rpy="${PI/2} 0 0"/>
-        <geometry>
-          <cylinder radius="${wheel_radius}" length="${wheel_width}"/>
+        <origin xyz="0 0 0" rpy="${PI/2} 0 0" />
+        <geometry>
+          <cylinder radius="${wheel_radius}" length="${wheel_width}" />
         </geometry>
       </collision>
       <inertial>
-        <origin xyz="0 0 0" rpy="0 0 0"/>
-        <mass value="0.477"/>
+        <origin xyz="0 0 0" rpy="0 0 0" />
+        <mass value="0.477" />
         <inertia
           ixx="0.0013" ixy="0" ixz="0"
           iyy="0.0024" iyz="0"
-          izz="0.0013"/>
+          izz="0.0013" />
       </inertial>
     </link>
@@ -49,12 +57,12 @@
       <material>Gazebo/DarkGrey</material>
       <selfCollide>false</selfCollide>
-      <mu1 value="0.5"/>
-      <mu2 value="0.5"/>
+      <mu1 value="0.5" />
+      <mu2 value="0.5" />
       <kp value="10000000.0" />
       <kd value="1" />
-      <fdir1 value="1 0 0"/>
+      <fdir1 value="1 0 0" />
     </gazebo>
     <joint name="${prefix}_wheel_joint" type="continuous">
-      <parent link="chassis_link"/>
+      <parent link="chassis_link" />
       <child link="${prefix}_wheel_link" />
       <xacro:insert_block name="joint_pose" />
@@ -88,31 +96,31 @@
   <joint name="base_link_joint" type="fixed">
     <origin xyz="0 0 0" rpy="0 0 0" />
-    <parent link="base_link"/>
+    <parent link="base_link" />
     <child link="chassis_link" />
   </joint>
   <link name="chassis_link">
     <visual>
-      <origin xyz="0 0 ${footprint_vertical_offset}" rpy="${PI/2} 0 ${PI/2}"/>
+      <origin xyz="0 0 ${footprint_vertical_offset}" rpy="${PI/2} 0 ${PI/2}" />
       <geometry>
-        <mesh filename="package://jackal_description/meshes/jackal-base.stl"/>
+        <mesh filename="package://jackal_description/meshes/jackal-base.stl" />
       </geometry>
       <material name="dark_grey" />
     </visual>
     <collision>
-      <origin xyz="0 0 ${chassis_height/2}"/>
+      <origin xyz="0 0 ${chassis_height/2}" />
       <geometry>
-        <box size="${chassis_length} ${chassis_width} ${chassis_height}"/>
+        <box size="${chassis_length} ${chassis_width} ${chassis_height}" />
       </geometry>
     </collision>
     <inertial>
       <!-- Center of mass -->
-      <origin xyz="0.012  0.002 0.067" rpy="0 0 0"/>
-      <mass value="16.523"/>
+      <origin xyz="0.012  0.002 0.067" rpy="0 0 0" />
+      <mass value="16.523" />
       <!-- Moments of inertia: ( chassis without wheels ) -->
       <inertia
         ixx="0.3136" ixy="-0.0008" ixz="0.0164"
         iyy="0.3922" iyz="-0.0009"
-        izz="0.4485"/>
-      </inertial>
+        izz="0.4485" />
+    </inertial>
   </link>
   <xacro:unless value="$(optenv JACKAL_FRONT_ACCESSORY_FENDER 0)">
@@ -120,5 +128,5 @@
       <visual>
         <geometry>
-          <mesh filename="package://jackal_description/meshes/jackal-fender.stl"/>
+          <mesh filename="package://jackal_description/meshes/jackal-fender.stl" />
         </geometry>
         <material name="yellow" />
@@ -130,10 +138,10 @@
       <visual>
         <geometry>
-          <mesh filename="package://jackal_description/meshes/accessory_fender.stl"/>
-        </geometry>
-        <material name="yellow" />
-      </visual>
-    </link>
-    <link name="front_fender_accessory_link"/>
+          <mesh filename="package://jackal_description/meshes/accessory_fender.stl" />
+        </geometry>
+        <material name="yellow" />
+      </visual>
+    </link>
+    <link name="front_fender_accessory_link" />
     <joint name="front_fender_accessory_joint" type="fixed">
       <origin xyz="0.25629 0 0.07455" rpy="${PI} 0 0" />
@@ -143,5 +151,5 @@
   </xacro:if>
   <joint name="front_fender_joint" type="fixed">
-    <origin xyz="0 0 0" rpy="0 0 0"/>
+    <origin xyz="0 0 0" rpy="0 0 0" />
     <parent link="chassis_link" />
     <child link="front_fender_link" />
@@ -151,5 +159,5 @@
       <visual>
         <geometry>
-          <mesh filename="package://jackal_description/meshes/jackal-fender.stl"/>
+          <mesh filename="package://jackal_description/meshes/jackal-fender.stl" />
         </geometry>
         <material name="yellow" />
@@ -161,10 +169,10 @@
       <visual>
         <geometry>
-          <mesh filename="package://jackal_description/meshes/accessory_fender.stl"/>
-        </geometry>
-        <material name="yellow" />
-      </visual>
-    </link>
-    <link name="rear_fender_accessory_link"/>
+          <mesh filename="package://jackal_description/meshes/accessory_fender.stl" />
+        </geometry>
+        <material name="yellow" />
+      </visual>
+    </link>
+    <link name="rear_fender_accessory_link" />
     <joint name="rear_fender_accessory_joint" type="fixed">
       <origin xyz="0.25629 0 0.07455" rpy="${PI} 0 0" />
@@ -174,5 +182,5 @@
   </xacro:if>
   <joint name="rear_fender_joint" type="fixed">
-    <origin xyz="0 0 0" rpy="0 0 ${PI}"/>
+    <origin xyz="0 0 0" rpy="0 0 ${PI}" />
     <parent link="chassis_link" />
     <child link="rear_fender_link" />
@@ -184,7 +192,8 @@
   <link name="imu_link">
     <inertial>
-      <mass value="0.001"/>
-      <origin xyz="0 0 0" rpy="0 0 0"/>
-      <inertia ixx="${dummy_inertia}" ixy="0.0" ixz="0.0" iyy="${dummy_inertia}" iyz="0.0" izz="${dummy_inertia}"/>
+      <mass value="0.001" />
+      <origin xyz="0 0 0" rpy="0 0 0" />
+      <inertia ixx="${dummy_inertia}" ixy="0.0" ixz="0.0" iyy="${dummy_inertia}" iyz="0.0"
+        izz="${dummy_inertia}" />
     </inertial>
   </link>
@@ -230,10 +239,10 @@
     <hardware>
       <xacro:if value="$(arg isaac_sim)">
-            <plugin>topic_based_ros2_control/TopicBasedSystem</plugin>
-            <param name="joint_commands_topic">/isaac_joint_commands</param>
-            <param name="joint_states_topic">/isaac_joint_states</param>
+        <plugin>topic_based_ros2_control/TopicBasedSystem</plugin>
+        <param name="joint_commands_topic">/isaac_joint_commands</param>
+        <param name="joint_states_topic">/isaac_joint_states</param>
       </xacro:if>
       <xacro:if value="$(arg gazebo_sim)">
-            <plugin>gazebo_ros2_control/GazeboSystem</plugin>
+        <plugin>gazebo_ros2_control/GazeboSystem</plugin>
       </xacro:if>
       <xacro:unless value="${$(arg gazebo_sim) or $(arg isaac_sim)}">
@@ -243,22 +252,22 @@
     </hardware>
     <joint name="front_left_wheel_joint">
-      <command_interface name="velocity"/>
-      <state_interface name="position"/>
-      <state_interface name="velocity"/>
+      <command_interface name="velocity" />
+      <state_interface name="position" />
+      <state_interface name="velocity" />
     </joint>
     <joint name="rear_left_wheel_joint">
-      <command_interface name="velocity"/>
-      <state_interface name="position"/>
-      <state_interface name="velocity"/>
+      <command_interface name="velocity" />
+      <state_interface name="position" />
+      <state_interface name="velocity" />
     </joint>
     <joint name="front_right_wheel_joint">
-      <command_interface name="velocity"/>
-      <state_interface name="position"/>
-      <state_interface name="velocity"/>
+      <command_interface name="velocity" />
+      <state_interface name="position" />
+      <state_interface name="velocity" />
     </joint>
     <joint name="rear_right_wheel_joint">
-      <command_interface name="velocity"/>
-      <state_interface name="position"/>
-      <state_interface name="velocity"/>
+      <command_interface name="velocity" />
+      <state_interface name="position" />
+      <state_interface name="velocity" />
     </joint>
   </ros2_control>
